Commit message: Fix P04

File: loader/description/urdf/loader.urdf (robot description, URDF)
Before this commit: robot loader, 18 links, 17 joints
Joints:
- joint Cat_982XE_P04_Joint: origin xyz=0.120276 0.0 2.31127 rpy=0 0 0 -> xyz=0.83742 0.0 0.97936 rpy=0 0 0; parent Cat_982XE_P01 -> Cat_982XE_P02

File: loader/description/urdf/loader.xacro (robot description, xacro)
@@ -66,6 +66,6 @@
     </link>
     <joint name="${prefix}P04_Joint" type="fixed">
-      <origin xyz="0.120276 0.0 2.31127" rpy="0 0 0" />
-      <parent link="${prefix}P01" />
+      <origin xyz="0.83742 0.0 0.97936" rpy="0 0 0" />
+      <parent link="${prefix}P02" />
       <child link="${prefix}P04" />
     </joint>

Commit message: Fix wheels

File: loader/description/urdf/loader.urdf (robot description, URDF)
Before this commit: robot loader, 18 links, 17 joints
Joints:
- joint Cat_982XE_P015_Joint: origin xyz=0.0 0.0 0.0 rpy=0 0 0 -> xyz=0.0 1.4457 0.0 rpy=0 0 0
- joint Cat_982XE_P016_Joint: origin xyz=0.0 0.0 0.0 rpy=0 0 0 -> xyz=0.0 -1.4457 0.0 rpy=0 0 0
- joint Cat_982XE_P018_Joint: origin xyz=1.8549 0.0 -0.39222 rpy=0 0 0 -> xyz=1.8549 1.4457 -0.39222 rpy=0 0 0
- joint Cat_982XE_P019_Joint: origin xyz=1.8549 0.0 -0.39222 rpy=0 0 0 -> xyz=1.8549 -1.4457 -0.39222 rpy=0 0 0

File: loader/description/urdf/loader.xacro (robot description, xacro)
@@ -336,5 +336,5 @@
     </link>
     <joint name="${prefix}P015_Joint" type="continuous">
-      <origin xyz="0.0 0.0 0.0" rpy="0 0 0" />
+      <origin xyz="0.0 1.4457 0.0" rpy="0 0 0" />
       <parent link="${prefix}P14" />
       <child link="${prefix}P15" />
@@ -348,5 +348,5 @@
       </visual>
       <collision>
-        <origin xyz="0.0 1.34357 0.0" rpy="${90*pi/180} 0 0" />
+        <origin xyz="0.0 -0.10213 0.0" rpy="${90*pi/180} 0 0" />
         <geometry>
           <cylinder radius="0.934162" length="0.817806" />
@@ -359,5 +359,5 @@
     </link>
     <joint name="${prefix}P016_Joint" type="continuous">
-      <origin xyz="0.0 0.0 0.0" rpy="0 0 0" />
+      <origin xyz="0.0 -1.4457 0.0" rpy="0 0 0" />
       <parent link="${prefix}P14" />
       <child link="${prefix}P16" />
@@ -371,5 +371,5 @@
       </visual>
       <collision>
-        <origin xyz="0.0 -1.34357 0.0" rpy="${90*pi/180} 0 0" />
+        <origin xyz="0.0 0.10213 0.0" rpy="${90*pi/180} 0 0" />
         <geometry>
           <cylinder radius="0.934162" length="0.817806" />
@@ -382,5 +382,5 @@
     </link>
     <joint name="${prefix}P018_Joint" type="continuous">
-      <origin xyz="1.8549 0.0 -0.39222" rpy="0 0 0" />
+      <origin xyz="1.8549 1.4457 -0.39222" rpy="0 0 0" />
       <parent link="${prefix}P02" />
       <child link="${prefix}P18" />
@@ -394,5 +394,5 @@
       </visual>
       <collision>
-        <origin xyz="0.0 1.34357 0.0" rpy="${90*pi/180} 0 0" />
+        <origin xyz="0.0 -0.10213 0.0" rpy="${90*pi/180} 0 0" />
         <geometry>
           <cylinder radius="0.934162" length="0.817806" />
@@ -405,5 +405,5 @@
     </link>
     <joint name="${prefix}P019_Joint" type="continuous">
-      <origin xyz="1.8549 0.0 -0.39222" rpy="0 0 0" />
+      <origin xyz="1.8549 -1.4457 -0.39222" rpy="0 0 0" />
       <parent link="${prefix}P02" />
       <child link="${prefix}P19" />
@@ -417,5 +417,5 @@
       </visual>
       <collision>
-        <origin xyz="0.0 -1.34357 0.0" rpy="${90*pi/180} 0 0" />
+        <origin xyz="0.0 0.10213 0.0" rpy="${90*pi/180} 0 0" />
         <geometry>
           <cylinder radius="0.934162" length="0.817806" />
