Commit message: Rename caterpillar to haul_truck

File: haul_truck/description/urdf/haul_truck.xacro (robot description, xacro)
@@ -1,10 +1,10 @@
 <?xml version="1.0" encoding="utf-8"?>
-<robot xmlns:xacro="http://www.ros.org/wiki/xacro" name="caterpillar">
-  <xacro:macro name="caterpillar" params="prefix:=''">
+<robot xmlns:xacro="http://www.ros.org/wiki/xacro" name="haul_truck">
+  <xacro:macro name="haul_truck" params="prefix:=''">
     <link name="${prefix}Main">
       <visual>
         <origin xyz="5.98719 0.0 3.1686" rpy="0 0 0" />
         <geometry>
-          <mesh filename="package://construction_vehicles/caterpillar/description/meshes/visual/Main.dae" />
+          <mesh filename="package://construction_vehicles/haul_truck/description/meshes/visual/Main.dae" />
         </geometry>
       </visual>
@@ -20,5 +20,5 @@
       <visual>
         <geometry>
-          <mesh filename="package://construction_vehicles/caterpillar/description/meshes/visual/FrontLeftSwivel.dae" />
+          <mesh filename="package://construction_vehicles/haul_truck/description/meshes/visual/FrontLeftSwivel.dae" />
         </geometry>
       </visual>
@@ -33,5 +33,5 @@
       <visual>
         <geometry>
-          <mesh filename="package://construction_vehicles/caterpillar/description/meshes/visual/FrontLeftWheel.dae" />
+          <mesh filename="package://construction_vehicles/haul_truck/description/meshes/visual/FrontLeftWheel.dae" />
         </geometry>
       </visual>
@@ -47,5 +47,5 @@
       <visual>
         <geometry>
-          <mesh filename="package://construction_vehicles/caterpillar/description/meshes/visual/FrontRightSwivel.dae" />
+          <mesh filename="package://construction_vehicles/haul_truck/description/meshes/visual/FrontRightSwivel.dae" />
         </geometry>
       </visual>
@@ -60,5 +60,5 @@
       <visual>
         <geometry>
-          <mesh filename="package://construction_vehicles/caterpillar/description/meshes/visual/FrontRightWheel.dae" />
+          <mesh filename="package://construction_vehicles/haul_truck/description/meshes/visual/FrontRightWheel.dae" />
         </geometry>
       </visual>
@@ -73,5 +73,5 @@
       <visual>
         <geometry>
-          <mesh filename="package://construction_vehicles/caterpillar/description/meshes/visual/RearLeftWheel.dae" />
+          <mesh filename="package://construction_vehicles/haul_truck/description/meshes/visual/RearLeftWheel.dae" />
         </geometry>
       </visual>
@@ -86,5 +86,5 @@
       <visual>
         <geometry>
-          <mesh filename="package://construction_vehicles/caterpillar/description/meshes/visual/RearRightWheel.dae" />
+          <mesh filename="package://construction_vehicles/haul_truck/description/meshes/visual/RearRightWheel.dae" />
         </geometry>
       </visual>
@@ -99,5 +99,5 @@
       <visual>
         <geometry>
-          <mesh filename="package://construction_vehicles/caterpillar/description/meshes/visual/Push1.dae" />
+          <mesh filename="package://construction_vehicles/haul_truck/description/meshes/visual/Push1.dae" />
         </geometry>
       </visual>
@@ -113,5 +113,5 @@
       <visual>
         <geometry>
-          <mesh filename="package://construction_vehicles/caterpillar/description/meshes/visual/Push3.dae" />
+          <mesh filename="package://construction_vehicles/haul_truck/description/meshes/visual/Push3.dae" />
         </geometry>
       </visual>
@@ -126,5 +126,5 @@
       <visual>
         <geometry>
-          <mesh filename="package://construction_vehicles/caterpillar/description/meshes/visual/BackPart.dae" />
+          <mesh filename="package://construction_vehicles/haul_truck/description/meshes/visual/BackPart.dae" />
         </geometry>
       </visual>
@@ -138,5 +138,5 @@
       <visual>
         <geometry>
-          <mesh filename="package://construction_vehicles/caterpillar/description/meshes/visual/Cabin.dae" />
+          <mesh filename="package://construction_vehicles/haul_truck/description/meshes/visual/Cabin.dae" />
         </geometry>
       </visual>
@@ -150,5 +150,5 @@
       <visual>
         <geometry>
-          <mesh filename="package://construction_vehicles/caterpillar/description/meshes/visual/Chair.dae" />
+          <mesh filename="package://construction_vehicles/haul_truck/description/meshes/visual/Chair.dae" />
         </geometry>
       </visual>
@@ -162,5 +162,5 @@
       <visual>
         <geometry>
-          <mesh filename="package://construction_vehicles/caterpillar/description/meshes/visual/Cockpit.dae" />
+          <mesh filename="package://construction_vehicles/haul_truck/description/meshes/visual/Cockpit.dae" />
         </geometry>
       </visual>
@@ -176,5 +176,5 @@
       <visual>
         <geometry>
-          <mesh filename="package://construction_vehicles/caterpillar/description/meshes/visual/DoorRight.dae" />
+          <mesh filename="package://construction_vehicles/haul_truck/description/meshes/visual/DoorRight.dae" />
         </geometry>
       </visual>
@@ -190,5 +190,5 @@
       <visual>
         <geometry>
-          <mesh filename="package://construction_vehicles/caterpillar/description/meshes/visual/DoorLeft.dae" />
+          <mesh filename="package://construction_vehicles/haul_truck/description/meshes/visual/DoorLeft.dae" />
         </geometry>
       </visual>
