Commit message: Update control

File: dump_truck/description/urdf/dump_truck.urdf (robot description, URDF)
Before this commit: robot dump_truck, 18 links, 17 joints
Links:
- added link Cat_740_DumperHolder; visual mesh filename=package://construction_vehicles/dump_truck/description/mesh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
- added link Cat_740_DumperPistonHeadLeft; visual mesh filename=package://construction_vehicles/dump_truck/description/mesh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
- added link Cat_740_DumperPistonHeadRight; visual mesh filename=package://construction_vehicles/dump_truck/description/mesh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
Joints:
- removed joint Cat_740_DumperCylinderLeftJoint
- removed joint Cat_740_DumperCylinderRightJoint
- removed joint Cat_740_DumperJoint
- removed joint Cat_740_DumperPistonLeftJoint
- removed joint Cat_740_DumperPistonRightJoint
- removed joint Cat_740_HeadJoint
- removed joint Cat_740_HeadTiltJoint
- removed joint Cat_740_SteeringCylinderLeftJoint
- removed joint Cat_740_SteeringCylinderRightJoint
- removed joint Cat_740_SteeringPistonLeftJoint
- removed joint Cat_740_SteeringPistonRightJoint
- removed joint Cat_740_WheelFrontLeftJoint
- removed joint Cat_740_WheelFrontRightJoint
- removed joint Cat_740_WheelRear1LeftJoint
- removed joint Cat_740_WheelRear1RightJoint
- removed joint Cat_740_WheelRear2LeftJoint
- removed joint Cat_740_WheelRear2RightJoint
- added joint Cat_740_DumperCylinderLeft_Joint: type continuous, parent Cat_740_DumperHolder, child Cat_740_DumperCylinderLeft, origin xyz=-0.013 0.509 -0.008 rpy=-0.1009 0.405 -0.311, axis 0 0 1
- added joint Cat_740_DumperCylinderRight_Joint: type continuous, parent Cat_740_DumperHolder, child Cat_740_DumperCylinderRight, origin xyz=-0.013 -0.509 -0.008 rpy=0.1009 0.405 0.311, axis 0 0 1
- added joint Cat_740_DumperHolder_Joint: type continuous, parent Cat_740_DumperChassis, child Cat_740_DumperHolder, origin xyz=0.197641 0 1.27301 rpy=0 0 0, axis 0 1 0
- added joint Cat_740_DumperPistonHeadLeft_Joint: type continuous, parent Cat_740_DumperPistonLeft, child Cat_740_DumperPistonHeadLeft, origin xyz=0 0 0 rpy=0 0 0, axis 1 0 0
- added joint Cat_740_DumperPistonHeadRight_Joint: type continuous, parent Cat_740_DumperPistonRight, child Cat_740_DumperPistonHeadRight, origin xyz=0 0 0 rpy=0 0 0, axis 1 0 0
- added joint Cat_740_DumperPistonLeft_Joint: type prismatic, parent Cat_740_DumperCylinderLeft, child Cat_740_DumperPistonLeft, origin xyz=-3.0 0 0 rpy=0 0 0, axis -1 0 0, limit lower=0 upper=1.8 effort=1000.0 velocity=1000.0
- added joint Cat_740_DumperPistonRight_Joint: type prismatic, parent Cat_740_DumperCylinderRight, child Cat_740_DumperPistonRight, origin xyz=-3.0 0 0 rpy=0 0 0, axis -1 0 0, limit lower=0 upper=1.8 effort=1000.0 velocity=1000.0
- added joint Cat_740_Dumper_Joint: type continuous, parent Cat_740_DumperChassis, child Cat_740_Dumper, origin xyz=-4.26 0 1.555 rpy=0 0 0, axis 0 -1 0
- added joint Cat_740_HeadTilt_Joint: type continuous, parent Cat_740_DumperChassis, child Cat_740_HeadTilt, origin xyz=0 0 1.186 rpy=0 0 0, axis 1 0 0
- added joint Cat_740_Head_Joint: type revolute, parent Cat_740_HeadTilt, child Cat_740_Head, origin xyz=0.8543 0 0 rpy=0 0 0, axis 0 0 1, limit lower=-0.7853981633974483 upper=0.7853981633974483 effort=1000.0 velocity=1000.0
- added joint Cat_740_SteeringCylinderLeft_Joint: type continuous, parent Cat_740_Head, child Cat_740_SteeringCylinderLeft, origin xyz=0.788 0.425 0.020 rpy=0 0 0, axis 0 0 1
- added joint Cat_740_SteeringCylinderRight_Joint: type continuous, parent Cat_740_Head, child Cat_740_SteeringCylinderRight, origin xyz=0.788 -0.425 0.020 rpy=0 0 0, axis 0 0 1
- added joint Cat_740_SteeringPistonLeft_Joint: type continuous, parent Cat_740_HeadTilt, child Cat_740_SteeringPistonLeft, origin xyz=0.560 0.426 0.022 rpy=0 0 0, axis 0 0 1
- added joint Cat_740_SteeringPistonRight_Joint: type continuous, parent Cat_740_HeadTilt, child Cat_740_SteeringPistonRight, origin xyz=0.560 -0.426 0.022 rpy=0 0 0, axis 0 0 1
- added joint Cat_740_WheelFrontLeft_Joint: type continuous, parent Cat_740_Head, child Cat_740_WheelFrontLeft, origin xyz=1.366 1.169 -0.297 rpy=0 0 0, axis 0 1 0
- added joint Cat_740_WheelFrontRight_Joint: type continuous, parent Cat_740_Head, child Cat_740_WheelFrontRight, origin xyz=1.366 -1.169 -0.297 rpy=0 0 0, axis 0 1 0
- added joint Cat_740_WheelRear1Left_Joint: type continuous, parent Cat_740_DumperChassis, child Cat_740_WheelRear1Left, origin xyz=-2.03074 1.169 0.889 rpy=0 0 0, axis 0 1 0
- added joint Cat_740_WheelRear1Right_Joint: type continuous, parent Cat_740_DumperChassis, child Cat_740_WheelRear1Right, origin xyz=-2.03074 -1.169 0.889 rpy=0 0 0, axis 0 1 0
- added joint Cat_740_WheelRear2Left_Joint: type continuous, parent Cat_740_DumperChassis, child Cat_740_WheelRear2Left, origin xyz=-3.99134 1.169 0.889 rpy=0 0 0, axis 0 1 0
- added joint Cat_740_WheelRear2Right_Joint: type continuous, parent Cat_740_DumperChassis, child Cat_740_WheelRear2Right, origin xyz=-3.99134 -1.169 0.889 rpy=0 0 0, axis 0 1 0

File: dump_truck/description/urdf/dump_truck.xacro (robot description, xacro)
@@ -10,5 +10,5 @@
       </visual>
     </link>
-    <joint name="${prefix}WheelRear1LeftJoint" type="continuous">
+    <joint name="${prefix}WheelRear1Left_Joint" type="continuous">
       <origin xyz="-2.03074 1.169 0.889" rpy="0 0 0" />
       <parent link="${prefix}DumperChassis" />
@@ -23,5 +23,5 @@
       </visual>
     </link>
-    <joint name="${prefix}WheelRear1RightJoint" type="continuous">
+    <joint name="${prefix}WheelRear1Right_Joint" type="continuous">
       <origin xyz="-2.03074 -1.169 0.889" rpy="0 0 0" />
       <parent link="${prefix}DumperChassis" />
@@ -36,5 +36,5 @@
       </visual>
     </link>
-    <joint name="${prefix}WheelRear2LeftJoint" type="continuous">
+    <joint name="${prefix}WheelRear2Left_Joint" type="continuous">
       <origin xyz="-3.99134 1.169 0.889" rpy="0 0 0" />
       <parent link="${prefix}DumperChassis" />
@@ -49,5 +49,5 @@
       </visual>
     </link>
-    <joint name="${prefix}WheelRear2RightJoint" type="continuous">
+    <joint name="${prefix}WheelRear2Right_Joint" type="continuous">
       <origin xyz="-3.99134 -1.169 0.889" rpy="0 0 0" />
       <parent link="${prefix}DumperChassis" />
@@ -62,5 +62,5 @@
       </visual>
     </link>
-    <joint name="${prefix}DumperJoint" type="continuous">
+    <joint name="${prefix}Dumper_Joint" type="continuous">
       <origin xyz="-4.26 0 1.555" rpy="0 0 0" />
       <parent link="${prefix}DumperChassis" />
@@ -75,7 +75,20 @@
       </visual>
     </link>
-    <joint name="${prefix}DumperCylinderLeftJoint" type="continuous">
-      <origin xyz="0.185013 0.508895 1.26466" rpy="-0.1009 0.405 -0.311" />
-      <parent link="${prefix}DumperChassis" />
+    <joint name="${prefix}DumperHolder_Joint" type="continuous">
+      <origin xyz="0.197641 0 1.27301" rpy="0 0 0" />
+      <parent link="${prefix}DumperChassis" />
+      <child link="${prefix}DumperHolder" />
+      <axis xyz="0 1 0" />
+    </joint>
+    <link name="${prefix}DumperHolder">
+      <visual>
+        <geometry>
+          <mesh filename="package://construction_vehicles/dump_truck/description/meshes/visual/DumperHolder.dae" />
+        </geometry>
+      </visual>
+    </link>
+    <joint name="${prefix}DumperCylinderLeft_Joint" type="continuous">
+      <origin xyz="-0.013 0.509 -0.008" rpy="-0.1009 0.405 -0.311" />
+      <parent link="${prefix}DumperHolder" />
       <child link="${prefix}DumperCylinderLeft" />
       <axis xyz="0 0 1" />
@@ -88,5 +101,5 @@
       </visual>
     </link>
-    <joint name="${prefix}DumperPistonLeftJoint" type="prismatic">
+    <joint name="${prefix}DumperPistonLeft_Joint" type="prismatic">
       <origin xyz="-3.0 0 0" rpy="0 0 0" />
       <parent link="${prefix}DumperCylinderLeft" />
@@ -102,7 +115,20 @@
       </visual>
     </link>
-    <joint name="${prefix}DumperCylinderRightJoint" type="continuous">
-      <origin xyz="0.185013 -0.508895 1.26466" rpy="0.1009 0.405 0.311" />
-      <parent link="${prefix}DumperChassis" />
+    <joint name="${prefix}DumperPistonHeadLeft_Joint" type="continuous">
+      <origin xyz="0 0 0" rpy="0 0 0" />
+      <parent link="${prefix}DumperPistonLeft" />
+      <child link="${prefix}DumperPistonHeadLeft" />
+      <axis xyz="1 0 0" />
+    </joint>
+    <link name="${prefix}DumperPistonHeadLeft">
+      <visual>
+        <geometry>
+          <mesh filename="package://construction_vehicles/dump_truck/description/meshes/visual/DumperPistonHead.dae" />
+        </geometry>
+      </visual>
+    </link>
+    <joint name="${prefix}DumperCylinderRight_Joint" type="continuous">
+      <origin xyz="-0.013 -0.509 -0.008" rpy="0.1009 0.405 0.311" />
+      <parent link="${prefix}DumperHolder" />
       <child link="${prefix}DumperCylinderRight" />
       <axis xyz="0 0 1" />
@@ -115,5 +141,5 @@
       </visual>
     </link>
-    <joint name="${prefix}DumperPistonRightJoint" type="prismatic">
+    <joint name="${prefix}DumperPistonRight_Joint" type="prismatic">
       <origin xyz="-3.0 0 0" rpy="0 0 0" />
       <parent link="${prefix}DumperCylinderRight" />
@@ -129,5 +155,18 @@
       </visual>
     </link>
-    <joint name="${prefix}SteeringPistonLeftJoint" type="continuous">
+    <joint name="${prefix}DumperPistonHeadRight_Joint" type="continuous">
+      <origin xyz="0 0 0" rpy="0 0 0" />
+      <parent link="${prefix}DumperPistonRight" />
+      <child link="${prefix}DumperPistonHeadRight" />
+      <axis xyz="1 0 0" />
+    </joint>
+    <link name="${prefix}DumperPistonHeadRight">
+      <visual>
+        <geometry>
+          <mesh filename="package://construction_vehicles/dump_truck/description/meshes/visual/DumperPistonHead.dae" />
+        </geometry>
+      </visual>
+    </link>
+    <joint name="${prefix}SteeringPistonLeft_Joint" type="continuous">
       <origin xyz="0.560 0.426 0.022" rpy="0 0 0" />
       <parent link="${prefix}HeadTilt" />
@@ -142,5 +181,5 @@
       </visual>
     </link>
-    <joint name="${prefix}SteeringPistonRightJoint" type="continuous">
+    <joint name="${prefix}SteeringPistonRight_Joint" type="continuous">
       <origin xyz="0.560 -0.426 0.022" rpy="0 0 0" />
       <parent link="${prefix}HeadTilt" />
@@ -155,5 +194,5 @@
       </visual>
     </link>
-    <joint name="${prefix}HeadTiltJoint" type="continuous">
+    <joint name="${prefix}HeadTilt_Joint" type="continuous">
       <origin xyz="0 0 1.186" rpy="0 0 0" />
       <parent link="${prefix}DumperChassis" />
@@ -168,5 +207,5 @@
       </visual>
     </link>
-    <joint name="${prefix}HeadJoint" type="revolute">
+    <joint name="${prefix}Head_Joint" type="revolute">
       <origin xyz="0.8543 0 0" rpy="0 0 0" />
       <parent link="${prefix}HeadTilt" />
@@ -182,5 +221,5 @@
       </visual>
     </link>
-    <joint name="${prefix}WheelFrontLeftJoint" type="continuous">
+    <joint name="${prefix}WheelFrontLeft_Joint" type="continuous">
       <origin xyz="1.366 1.169 -0.297" rpy="0 0 0" />
       <parent link="${prefix}Head" />
@@ -195,5 +234,5 @@
       </visual>
     </link>
-    <joint name="${prefix}WheelFrontRightJoint" type="continuous">
+    <joint name="${prefix}WheelFrontRight_Joint" type="continuous">
       <origin xyz="1.366 -1.169 -0.297" rpy="0 0 0" />
       <parent link="${prefix}Head" />
@@ -208,5 +247,5 @@
       </visual>
     </link>
-    <joint name="${prefix}SteeringCylinderLeftJoint" type="continuous">
+    <joint name="${prefix}SteeringCylinderLeft_Joint" type="continuous">
       <origin xyz="0.788 0.425 0.020" rpy="0 0 0" />
       <parent link="${prefix}Head" />
@@ -221,5 +260,5 @@
       </visual>
     </link>
-    <joint name="${prefix}SteeringCylinderRightJoint" type="continuous">
+    <joint name="${prefix}SteeringCylinderRight_Joint" type="continuous">
       <origin xyz="0.788 -0.425 0.020" rpy="0 0 0" />
       <parent link="${prefix}Head" />
