Commit message: Fix excavator

File: excavator/description/urdf/excavator.urdf (robot description, URDF)
Before this commit: robot excavator, 20 links, 19 joints
Links:
- removed link Cat_395_Boom_Cylinder_Left_1
- removed link Cat_395_Boom_Cylinder_Left_2
- removed link Cat_395_Boom_Cylinder_Right_1
- removed link Cat_395_Boom_Cylinder_Right_2
- added link Cat_395_Boom_Cylinder_1, mass 1000.0; collision cylinder length=2.46036 radius=0.271748; collision cylinder length=2.46036 radius=0.271748
- added link Cat_395_Boom_Cylinder_2, mass 1000.0; collision cylinder length=2.46738 radius=0.120975; collision cylinder length=2.46738 radius=0.120975
- added link Cat_395_Wheel_Left, mass 1000.0; collision cylinder length=0.177212 radius=0.46; visual mesh filename=package://construction_vehicles/excavator/description/meshe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
- added link Cat_395_Wheel_Right, mass 1000.0; collision cylinder length=0.177212 radius=0.46; visual mesh filename=package://construction_vehicles/excavator/description/meshe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
Joints:
- removed joint Cat_395_Boom_Cylinder_Left_1_Joint
- removed joint Cat_395_Boom_Cylinder_Left_2_Joint
- removed joint Cat_395_Boom_Cylinder_Right_1_Joint
- removed joint Cat_395_Boom_Cylinder_Right_2_Joint
- added joint Cat_395_Boom_Cylinder_1_Joint: type continuous, parent Cat_395_Cabin, child Cat_395_Boom_Cylinder_1, origin xyz=-1.269 0.0 1.167 rpy=0 -0.593411945678072 0, axis 0 1 0
- added joint Cat_395_Boom_Cylinder_2_Joint: type prismatic, parent Cat_395_Boom_Cylinder_1, child Cat_395_Boom_Cylinder_2, origin xyz=0.0 0.0 4.13344 rpy=0 0 0, axis 0 0 1, limit lower=-1.70 upper=0.31 effort=1000.0 velocity=1000.0
- added joint Cat_395_Wheel_Left_Joint: type continuous, parent Cat_395_Base, child Cat_395_Wheel_Left, origin xyz=-2.65099 -1.70966 0.707697 rpy=1.5707963267948966 0 0, axis 0 0 1
- added joint Cat_395_Wheel_Right_Joint: type continuous, parent Cat_395_Base, child Cat_395_Wheel_Right, origin xyz=-2.65099 1.70966 0.707697 rpy=1.5707963267948966 0 0, axis 0 0 1
- joint Cat_395_Bucket_Cylinder_1_Joint: origin xyz=-0.972 0.000 1.190 rpy=0 0.15655603390389136 0 -> xyz=-0.999 0.000 1.120 rpy=0 0.15655603390389136 0
- joint Cat_395_Motor_Right_Joint: origin xyz=2.56148 1.8052 0.707696 rpy=-1.5707963267948966 0 0 -> xyz=2.56148 1.8052 0.707696 rpy=1.5707963267948966 0 0
- joint Cat_395_Part_12_Joint: origin xyz=-0.719 0.000 0.036 rpy=0 0.069 0 -> xyz=-0.719 0.000 0.036 rpy=0 0 0

File: excavator/description/urdf/excavator.xacro (robot description, xacro)
@@ -6,5 +6,5 @@
         <origin xyz="0.0 0.0 0.793384" rpy="0 0 0" />
         <geometry>
-          <mesh filename="package://construction_vehicles/excavator/description/meshes/visual/Base.dae" />
+          <mesh filename="package://construction_vehicles/excavator/description/meshes/visual/Base_Without_Wheels.dae" />
         </geometry>
       </visual>
@@ -85,5 +85,5 @@
     </link>
     <joint name="${prefix}Motor_Right_Joint" type="continuous">
-      <origin xyz="2.56148 1.8052 0.707696" rpy="${-pi/2} 0 0" />
+      <origin xyz="2.56148 1.8052 0.707696" rpy="${pi/2} 0 0" />
       <parent link="${prefix}Base" />
       <child link="${prefix}Motor_Right" />
@@ -92,4 +92,5 @@
     <link name="${prefix}Motor_Right">
       <visual>
+        <origin xyz="0 0 0" rpy="${pi} 0 0" />
         <geometry>
           <mesh filename="package://construction_vehicles/excavator/description/meshes/visual/Motor.dae" />
@@ -99,4 +100,48 @@
         <geometry>
           <cylinder radius="0.522574" length="0.531622" />
+        </geometry>
+      </collision>
+      <inertial>
+        <mass value="1000.0" />
+        <inertia ixx="100.0" ixy="0.0" ixz="0.0" iyy="100.0" iyz="0.0" izz="100.0" />
+      </inertial>
+    </link>
+    <joint name="${prefix}Wheel_Left_Joint" type="continuous">
+      <origin xyz="-2.65099 -1.70966 0.707697" rpy="${pi/2} 0 0" />
+      <parent link="${prefix}Base" />
+      <child link="${prefix}Wheel_Left" />
+      <axis xyz="0 0 1" />
+    </joint>
+    <link name="${prefix}Wheel_Left">
+      <visual>
+        <geometry>
+          <mesh filename="package://construction_vehicles/excavator/description/meshes/visual/Wheel.dae" />
+        </geometry>
+      </visual>
+      <collision>
+        <geometry>
+          <cylinder radius="0.46" length="0.177212" />
+        </geometry>
+      </collision>
+      <inertial>
+        <mass value="1000.0" />
+        <inertia ixx="100.0" ixy="0.0" ixz="0.0" iyy="100.0" iyz="0.0" izz="100.0" />
+      </inertial>
+    </link>
+    <joint name="${prefix}Wheel_Right_Joint" type="continuous">
+      <origin xyz="-2.65099 1.70966 0.707697" rpy="${pi/2} 0 0" />
+      <parent link="${prefix}Base" />
+      <child link="${prefix}Wheel_Right" />
+      <axis xyz="0 0 1" />
+    </joint>
+    <link name="${prefix}Wheel_Right">
+      <visual>
+        <geometry>
+          <mesh filename="package://construction_vehicles/excavator/description/meshes/visual/Wheel.dae" />
+        </geometry>
+      </visual>
+      <collision>
+        <geometry>
+          <cylinder radius="0.46" length="0.177212" />
         </geometry>
       </collision>
@@ -175,89 +220,68 @@
       </inertial>
     </link>
-    <joint name="${prefix}Boom_Cylinder_Left_1_Joint" type="continuous">
-      <origin xyz="-1.269 -0.506 1.167" rpy="0 ${-34/180 * pi} 0" />
+    <joint name="${prefix}Boom_Cylinder_1_Joint" type="continuous">
+      <origin xyz="-1.269 0.0 1.167" rpy="0 ${-34/180 * pi} 0" />
       <parent link="${prefix}Cabin" />
-      <child link="${prefix}Boom_Cylinder_Left_1" />
-      <axis xyz="0 1 0" />
-    </joint>
-    <link name="${prefix}Boom_Cylinder_Left_1">
-      <visual>
+      <child link="${prefix}Boom_Cylinder_1" />
+      <axis xyz="0 1 0" />
+    </joint>
+    <link name="${prefix}Boom_Cylinder_1">
+      <visual>
+        <origin xyz="0.0 -0.506 0.0" rpy="0 0 0" />
         <geometry>
           <mesh filename="package://construction_vehicles/excavator/description/meshes/visual/Boom_Cylinder_Left_1.dae" />
         </geometry>
       </visual>
-      <collision>
-        <origin xyz="0.0 0.0 1.09389" rpy="0 0 0" />
+      <visual>
+        <origin xyz="0.0 0.506 0.0" rpy="0 0 0" />
+        <geometry>
+          <mesh filename="package://construction_vehicles/excavator/description/meshes/visual/Boom_Cylinder_Right_1.dae" />
+        </geometry>
+      </visual>
+      <collision>
+        <origin xyz="0.0 -0.506 1.09389" rpy="0 0 0" />
         <geometry>
           <cylinder radius="0.271748" length="2.46036" />
         </geometry>
       </collision>
-      <inertial>
-        <mass value="1000.0" />
-        <inertia ixx="100.0" ixy="0.0" ixz="0.0" iyy="100.0" iyz="0.0" izz="100.0" />
-      </inertial>
-    </link>
-    <joint name="${prefix}Boom_Cylinder_Left_2_Joint" type="prismatic">
+      <collision>
+        <origin xyz="0.0 0.506 1.09389" rpy="0 0 0" />
+        <geometry>
+          <cylinder radius="0.271748" length="2.46036" />
+        </geometry>
+      </collision>
+      <inertial>
+        <mass value="1000.0" />
+        <inertia ixx="100.0" ixy="0.0" ixz="0.0" iyy="100.0" iyz="0.0" izz="100.0" />
+      </inertial>
+    </link>
+    <joint name="${prefix}Boom_Cylinder_2_Joint" type="prismatic">
       <origin xyz="0.0 0.0 4.13344" rpy="0 0 0" />
-      <parent link="${prefix}Boom_Cylinder_Left_1" />
-      <child link="${prefix}Boom_Cylinder_Left_2" />
+      <parent link="${prefix}Boom_Cylinder_1" />
+      <child link="${prefix}Boom_Cylinder_2" />
       <axis xyz="0 0 1" />
       <limit lower="-1.70" upper="0.31" effort="1000.0" velocity="1000.0" />
     </joint>
-    <link name="${prefix}Boom_Cylinder_Left_2">
-      <visual>
+    <link name="${prefix}Boom_Cylinder_2">
+      <visual>
+        <origin xyz="0.0 -0.506 0.0" rpy="0 0 0" />
         <geometry>
           <mesh filename="package://construction_vehicles/excavator/description/meshes/visual/Boom_Cylinder_Left_2.dae" />
         </geometry>
       </visual>
-      <collision>
-        <origin xyz="0.0 0.0 -1.11271" rpy="0 0 0" />
+      <visual>
+        <origin xyz="0.0 0.506 0.0" rpy="0 0 0" />
+        <geometry>
+          <mesh filename="package://construction_vehicles/excavator/description/meshes/visual/Boom_Cylinder_Right_2.dae" />
+        </geometry>
+      </visual>
+      <collision>
+        <origin xyz="0.0 -0.506 -1.11271" rpy="0 0 0" />
         <geometry>
           <cylinder radius="0.120975" length="2.46738" />
         </geometry>
       </collision>
-      <inertial>
-        <mass value="1000.0" />
-        <inertia ixx="100.0" ixy="0.0" ixz="0.0" iyy="100.0" iyz="0.0" izz="100.0" />
-      </inertial>
-    </link>
-    <joint name="${prefix}Boom_Cylinder_Right_1_Joint" type="continuous">
-      <origin xyz="-1.269 0.506 1.167" rpy="0 ${-34/180 * pi} 0" />
-      <parent link="${prefix}Cabin" />
-      <child link="${prefix}Boom_Cylinder_Right_1" />
-      <axis xyz="0 1 0" />
-    </joint>
-    <link name="${prefix}Boom_Cylinder_Right_1">
-      <visual>
-        <geometry>
-          <mesh filename="package://construction_vehicles/excavator/description/meshes/visual/Boom_Cylinder_Right_1.dae" />
-        </geometry>
-      </visual>
-      <collision>
-        <origin xyz="0.0 0.0 1.09389" rpy="0 0 0" />
-        <geometry>
-          <cylinder radius="0.271748" length="2.46036" />
-        </geometry>
-      </collision>
-      <inertial>
-        <mass value="1000.0" />
-        <inertia ixx="100.0" ixy="0.0" ixz="0.0" iyy="100.0" iyz="0.0" izz="100.0" />
-      </inertial>
-    </link>
-    <joint name="${prefix}Boom_Cylinder_Right_2_Joint" type="prismatic">
-      <origin xyz="0.0 0.0 4.13344" rpy="0 0 0" />
-      <parent link="${prefix}Boom_Cylinder_Right_1" />
-      <child link="${prefix}Boom_Cylinder_Right_2" />
-      <axis xyz="0 0 1" />
-      <limit lower="-1.70" upper="0.31" effort="1000.0" velocity="1000.0" />
-    </joint>
-    <link name="${prefix}Boom_Cylinder_Right_2">
-      <visual>
-        <geometry>
-          <mesh filename="package://construction_vehicles/excavator/description/meshes/visual/Boom_Cylinder_Right_2.dae" />
-        </geometry>
-      </visual>
-      <collision>
-        <origin xyz="0.0 0.0 -1.11271" rpy="0 0 0" />
+      <collision>
+        <origin xyz="0.0 0.506 -1.11271" rpy="0 0 0" />
         <geometry>
           <cylinder radius="0.120975" length="2.46738" />
@@ -339,5 +363,5 @@
     </link>
     <joint name="${prefix}Bucket_Cylinder_1_Joint" type="continuous">
-      <origin xyz="-0.972 0.000 1.190" rpy="0 ${8.97/180 * pi} 0" />
+      <origin xyz="-0.999 0.000 1.120" rpy="0 ${8.97/180 * pi} 0" />
       <parent link="${prefix}Arm" />
       <child link="${prefix}Bucket_Cylinder_1" />
@@ -430,5 +454,5 @@
     </link>
     <joint name="${prefix}Part_12_Joint" type="continuous">
-      <origin xyz="-0.719 0.000 0.036" rpy="0 0.069 0" />
+      <origin xyz="-0.719 0.000 0.036" rpy="0 0 0" />
       <parent link="${prefix}Bucket" />
       <child link="${prefix}Part_12" />

Commit message: Update

File: excavator/description/urdf/excavator.urdf (robot description, URDF)
Before this commit: robot excavator, 20 links, 19 joints
Links:
- link Cat_395_Arm: mass 1000.0 -> None
- link Cat_395_Arm_Cylinder_1: mass 1000.0 -> None
- link Cat_395_Arm_Cylinder_2: mass 1000.0 -> None
- link Cat_395_Base: mass 1000.0 -> None
- link Cat_395_Boom: mass 1000.0 -> None
- link Cat_395_Boom_Cylinder_1: mass 1000.0 -> None
- link Cat_395_Boom_Cylinder_2: mass 1000.0 -> None
- link Cat_395_Bucket: mass 1000.0 -> None
- link Cat_395_Bucket_Cylinder_1: mass 1000.0 -> None
- link Cat_395_Bucket_Cylinder_2: mass 1000.0 -> None
- link Cat_395_Cabin: mass 1000.0 -> None
- link Cat_395_Door: mass 1000.0 -> None
- link Cat_395_Motor_Left: mass 1000.0 -> None
- link Cat_395_Motor_Right: mass 1000.0 -> None
- link Cat_395_Part_11: mass 1000.0 -> None
- link Cat_395_Part_12: mass 1000.0 -> None
- link Cat_395_Track_Left: mass 1000.0 -> None
- link Cat_395_Track_Right: mass 1000.0 -> None
- link Cat_395_Wheel_Left: mass 1000.0 -> None
- link Cat_395_Wheel_Right: mass 1000.0 -> None
Joints:
- joint Cat_395_Motor_Left_Joint: axis 0 0 1 -> 0 -1 0; origin xyz=2.56148 -1.8052 0.707696 rpy=1.5707963267948966 0 0 -> xyz=2.56148 -1.8052 0.707696 rpy=0 0 0
- joint Cat_395_Motor_Right_Joint: axis 0 0 1 -> 0 -1 0; origin xyz=2.56148 1.8052 0.707696 rpy=1.5707963267948966 0 0 -> xyz=2.56148 1.8052 0.707696 rpy=0 0 0
- joint Cat_395_Wheel_Left_Joint: axis 0 0 1 -> 0 -1 0; origin xyz=-2.65099 -1.70966 0.707697 rpy=1.5707963267948966 0 0 -> xyz=-2.65099 -1.70966 0.707697 rpy=0 0 0
- joint Cat_395_Wheel_Right_Joint: axis 0 0 1 -> 0 -1 0; origin xyz=-2.65099 1.70966 0.707697 rpy=1.5707963267948966 0 0 -> xyz=-2.65099 1.70966 0.707697 rpy=0 0 0

File: excavator/description/urdf/excavator.xacro (robot description, xacro)
@@ -4,7 +4,7 @@
     <link name="${prefix}Base">
       <visual>
-        <origin xyz="0.0 0.0 0.793384" rpy="0 0 0" />
-        <geometry>
-          <mesh filename="package://construction_vehicles/excavator/description/meshes/visual/Base_Without_Wheels.dae" />
+        <origin xyz="0.0 0.0 0.793384" rpy="0 0 ${pi}" />
+        <geometry>
+          <mesh filename="package://construction_vehicles/excavator/description/meshes/visual/Base_Without_Wheels_Rotate_180.dae" />
         </geometry>
       </visual>
@@ -15,8 +15,4 @@
         </geometry>
       </collision>
-      <inertial>
-        <mass value="1000.0" />
-        <inertia ixx="100.0" ixy="0.0" ixz="0.0" iyy="100.0" iyz="0.0" izz="100.0" />
-      </inertial>
     </link>
     <joint name="${prefix}Track_Left_Joint" type="fixed">
@@ -36,8 +32,4 @@
         </geometry>
       </collision>
-      <inertial>
-        <mass value="1000.0" />
-        <inertia ixx="100.0" ixy="0.0" ixz="0.0" iyy="100.0" iyz="0.0" izz="100.0" />
-      </inertial>
     </link>
     <joint name="${prefix}Track_Right_Joint" type="fixed">
@@ -57,19 +49,15 @@
         </geometry>
       </collision>
-      <inertial>
-        <mass value="1000.0" />
-        <inertia ixx="100.0" ixy="0.0" ixz="0.0" iyy="100.0" iyz="0.0" izz="100.0" />
-      </inertial>
     </link>
     <joint name="${prefix}Motor_Left_Joint" type="continuous">
-      <origin xyz="2.56148 -1.8052 0.707696" rpy="${pi/2} 0 0" />
+      <origin xyz="2.56148 -1.8052 0.707696" rpy="0 0 0" />
       <parent link="${prefix}Base" />
       <child link="${prefix}Motor_Left" />
-      <axis xyz="0 0 1" />
+      <axis xyz="0 -1 0" />
     </joint>
     <link name="${prefix}Motor_Left">
       <visual>
         <geometry>
-          <mesh filename="package://construction_vehicles/excavator/description/meshes/visual/Motor.dae" />
+          <mesh filename="package://construction_vehicles/excavator/description/meshes/visual/Motor_Left.dae" />
         </geometry>
       </visual>
@@ -79,20 +67,15 @@
         </geometry>
       </collision>
-      <inertial>
-        <mass value="1000.0" />
-        <inertia ixx="100.0" ixy="0.0" ixz="0.0" iyy="100.0" iyz="0.0" izz="100.0" />
-      </inertial>
     </link>
     <joint name="${prefix}Motor_Right_Joint" type="continuous">
-      <origin xyz="2.56148 1.8052 0.707696" rpy="${pi/2} 0 0" />
+      <origin xyz="2.56148 1.8052 0.707696" rpy="0 0 0" />
       <parent link="${prefix}Base" />
       <child link="${prefix}Motor_Right" />
-      <axis xyz="0 0 1" />
+      <axis xyz="0 -1 0" />
     </joint>
     <link name="${prefix}Motor_Right">
       <visual>
-        <origin xyz="0 0 0" rpy="${pi} 0 0" />
-        <geometry>
-          <mesh filename="package://construction_vehicles/excavator/description/meshes/visual/Motor.dae" />
+        <geometry>
+          <mesh filename="package://construction_vehicles/excavator/description/meshes/visual/Motor_Right.dae" />
         </geometry>
       </visual>
@@ -102,14 +85,10 @@
         </geometry>
       </collision>
-      <inertial>
-        <mass value="1000.0" />
-        <inertia ixx="100.0" ixy="0.0" ixz="0.0" iyy="100.0" iyz="0.0" izz="100.0" />
-      </inertial>
     </link>
     <joint name="${prefix}Wheel_Left_Joint" type="continuous">
-      <origin xyz="-2.65099 -1.70966 0.707697" rpy="${pi/2} 0 0" />
+      <origin xyz="-2.65099 -1.70966 0.707697" rpy="0 0 0" />
       <parent link="${prefix}Base" />
       <child link="${prefix}Wheel_Left" />
-      <axis xyz="0 0 1" />
+      <axis xyz="0 -1 0" />
     </joint>
     <link name="${prefix}Wheel_Left">
@@ -124,14 +103,10 @@
         </geometry>
       </collision>
-      <inertial>
-        <mass value="1000.0" />
-        <inertia ixx="100.0" ixy="0.0" ixz="0.0" iyy="100.0" iyz="0.0" izz="100.0" />
-      </inertial>
     </link>
     <joint name="${prefix}Wheel_Right_Joint" type="continuous">
-      <origin xyz="-2.65099 1.70966 0.707697" rpy="${pi/2} 0 0" />
+      <origin xyz="-2.65099 1.70966 0.707697" rpy="0 0 0" />
       <parent link="${prefix}Base" />
       <child link="${prefix}Wheel_Right" />
-      <axis xyz="0 0 1" />
+      <axis xyz="0 -1 0" />
     </joint>
     <link name="${prefix}Wheel_Right">
@@ -146,8 +121,4 @@
         </geometry>
       </collision>
-      <inertial>
-        <mass value="1000.0" />
-        <inertia ixx="100.0" ixy="0.0" ixz="0.0" iyy="100.0" iyz="0.0" izz="100.0" />
-      </inertial>
     </link>
     <joint name="Cat_395_Cabin_Joint" type="revolute">
@@ -170,8 +141,4 @@
         </geometry>
       </collision>
-      <inertial>
-        <mass value="1000.0" />
-        <inertia ixx="100.0" ixy="0.0" ixz="0.0" iyy="100.0" iyz="0.0" izz="100.0" />
-      </inertial>
     </link>
     <joint name="${prefix}Door_Joint" type="revolute">
@@ -193,8 +160,4 @@
         </geometry>
       </collision>
-      <inertial>
-        <mass value="1000.0" />
-        <inertia ixx="100.0" ixy="0.0" ixz="0.0" iyy="100.0" iyz="0.0" izz="100.0" />
-      </inertial>
     </link>
     <joint name="${prefix}Boom_Joint" type="continuous">
@@ -215,8 +178,4 @@
         </geometry>
       </collision>
-      <inertial>
-        <mass value="1000.0" />
-        <inertia ixx="100.0" ixy="0.0" ixz="0.0" iyy="100.0" iyz="0.0" izz="100.0" />
-      </inertial>
     </link>
     <joint name="${prefix}Boom_Cylinder_1_Joint" type="continuous">
@@ -251,8 +210,4 @@
         </geometry>
       </collision>
-      <inertial>
-        <mass value="1000.0" />
-        <inertia ixx="100.0" ixy="0.0" ixz="0.0" iyy="100.0" iyz="0.0" izz="100.0" />
-      </inertial>
     </link>
     <joint name="${prefix}Boom_Cylinder_2_Joint" type="prismatic">
@@ -288,8 +243,4 @@
         </geometry>
       </collision>
-      <inertial>
-        <mass value="1000.0" />
-        <inertia ixx="100.0" ixy="0.0" ixz="0.0" iyy="100.0" iyz="0.0" izz="100.0" />
-      </inertial>
     </link>
     <joint name="${prefix}Arm_Cylinder_1_Joint" type="continuous">
@@ -311,8 +262,4 @@
         </geometry>
       </collision>
-      <inertial>
-        <mass value="1000.0" />
-        <inertia ixx="100.0" ixy="0.0" ixz="0.0" iyy="100.0" iyz="0.0" izz="100.0" />
-      </inertial>
     </link>
     <joint name="${prefix}Arm_Cylinder_2_Joint" type="prismatic">
@@ -335,8 +282,4 @@
         </geometry>
       </collision>
-      <inertial>
-        <mass value="1000.0" />
-        <inertia ixx="100.0" ixy="0.0" ixz="0.0" iyy="100.0" iyz="0.0" izz="100.0" />
-      </inertial>
     </link>
     <joint name="${prefix}Arm_Joint" type="continuous">
@@ -357,8 +300,4 @@
         </geometry>
       </collision>
-      <inertial>
-        <mass value="1000.0" />
-        <inertia ixx="100.0" ixy="0.0" ixz="0.0" iyy="100.0" iyz="0.0" izz="100.0" />
-      </inertial>
     </link>
     <joint name="${prefix}Bucket_Cylinder_1_Joint" type="continuous">
@@ -380,8 +319,4 @@
         </geometry>
       </collision>
-      <inertial>
-        <mass value="1000.0" />
-        <inertia ixx="100.0" ixy="0.0" ixz="0.0" iyy="100.0" iyz="0.0" izz="100.0" />
-      </inertial>
     </link>
     <joint name="${prefix}Bucket_Cylinder_2_Joint" type="prismatic">
@@ -404,8 +339,4 @@
         </geometry>
       </collision>
-      <inertial>
-        <mass value="1000.0" />
-        <inertia ixx="100.0" ixy="0.0" ixz="0.0" iyy="100.0" iyz="0.0" izz="100.0" />
-      </inertial>
     </link>
     <joint name="${prefix}Part_11_Joint" type="continuous">
@@ -426,8 +357,4 @@
         </geometry>
       </collision>
-      <inertial>
-        <mass value="1000.0" />
-        <inertia ixx="100.0" ixy="0.0" ixz="0.0" iyy="100.0" iyz="0.0" izz="100.0" />
-      </inertial>
     </link>
     <joint name="${prefix}Bucket_Joint" type="continuous">
@@ -448,8 +375,4 @@
         </geometry>
       </collision>
-      <inertial>
-        <mass value="1000.0" />
-        <inertia ixx="100.0" ixy="0.0" ixz="0.0" iyy="100.0" iyz="0.0" izz="100.0" />
-      </inertial>
     </link>
     <joint name="${prefix}Part_12_Joint" type="continuous">
@@ -470,8 +393,4 @@
         </geometry>
       </collision>
-      <inertial>
-        <mass value="1000.0" />
-        <inertia ixx="100.0" ixy="0.0" ixz="0.0" iyy="100.0" iyz="0.0" izz="100.0" />
-      </inertial>
     </link>
   </xacro:macro>
