Commit message: Fix excavator rotation and remove collision

File: excavator/description/urdf/excavator.urdf (robot description, URDF)
Before this commit: robot excavator, 20 links, 19 joints
Links:
- link Cat_395_Arm: geometry visual mesh filename=package://construction_vehicles/excavator/description/meshe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
- link Cat_395_Arm_Cylinder_1: geometry visual mesh filename=package://construction_vehicles/excavator/description/meshe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
- link Cat_395_Arm_Cylinder_2: geometry visual mesh filename=package://construction_vehicles/excavator/description/meshe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
- link Cat_395_Base: geometry visual mesh filename=package://construction_vehicles/excavator/description/meshe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
- link Cat_395_Boom: geometry visual mesh filename=package://construction_vehicles/excavator/description/meshe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
- link Cat_395_Boom_Cylinder_1: geometry visual mesh filename=package://construction_vehicles/excavator/description/meshe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; visual mesh filename=package://construction_vehicles/excavator/description/meshe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
- link Cat_395_Boom_Cylinder_2: geometry visual mesh filename=package://construction_vehicles/excavator/description/meshe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; visual mesh filename=package://construction_vehicles/excavator/description/meshe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
- link Cat_395_Bucket: geometry visual mesh filename=package://construction_vehicles/excavator/description/meshe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
- link Cat_395_Bucket_Cylinder_1: geometry visual mesh filename=package://construction_vehicles/excavator/description/meshe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
- link Cat_395_Bucket_Cylinder_2: geometry visual mesh filename=package://construction_vehicles/excavator/description/meshe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
- link Cat_395_Cabin: geometry visual mesh filename=package://construction_vehicles/excavator/description/meshe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
- link Cat_395_Door: geometry visual mesh filename=package://construction_vehicles/excavator/description/meshe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
- link Cat_395_Motor_Left: geometry visual mesh filename=package://construction_vehicles/excavator/description/meshe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
- link Cat_395_Motor_Right: geometry visual mesh filename=package://construction_vehicles/excavator/description/meshe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
- link Cat_395_Part_11: geometry visual mesh filename=package://construction_vehicles/excavator/description/meshe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
- link Cat_395_Part_12: geometry visual mesh filename=package://construction_vehicles/excavator/description/meshe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
- link Cat_395_Track_Left: geometry visual mesh filename=package://construction_vehicles/excavator/description/meshe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
- link Cat_395_Track_Right: geometry visual mesh filename=package://construction_vehicles/excavator/description/meshe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
- link Cat_395_Wheel_Left: geometry visual mesh filename=package://construction_vehicles/excavator/description/meshe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
- link Cat_395_Wheel_Right: geometry visual mesh filename=package://construction_vehicles/excavator/description/meshe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
Joints:
- joint Cat_395_Arm_Cylinder_1_Joint: origin xyz=-2.605 0.000 3.306 rpy=0 -1.413716694115407 0 -> xyz=2.605 0.000 3.306 rpy=0 1.413716694115407 0
- joint Cat_395_Arm_Joint: origin xyz=-7.002 0.000 2.732 rpy=0 0 0 -> xyz=7.002 0.000 2.732 rpy=0 0 0
- joint Cat_395_Boom_Cylinder_1_Joint: origin xyz=-1.269 0.0 1.167 rpy=0 -0.593411945678072 0 -> xyz=1.269 0.0 1.167 rpy=0 0.593411945678072 0
- joint Cat_395_Boom_Joint: origin xyz=-0.340 0.0 2.047 rpy=0 0 0 -> xyz=0.340 0.0 2.047 rpy=0 0 0
- joint Cat_395_Bucket_Cylinder_1_Joint: origin xyz=-0.999 0.000 1.120 rpy=0 0.15655603390389136 0 -> xyz=0.999 0.000 1.120 rpy=0 -0.15655603390389136 0
- joint Cat_395_Bucket_Joint: origin xyz=-0.659 0.000 -2.843 rpy=0 0 0 -> xyz=0.659 0.0 -2.843 rpy=0 0 0
- joint Cat_395_Door_Joint: origin xyz=-0.9692 -1.757323 2.610876 rpy=0 0 0 -> xyz=0.9692 1.757323 2.610876 rpy=0 0 0
- joint Cat_395_Motor_Left_Joint: origin xyz=2.56148 -1.8052 0.707696 rpy=0 0 0 -> xyz=-2.56148 1.8052 0.707696 rpy=0 0 0
- joint Cat_395_Motor_Right_Joint: origin xyz=2.56148 1.8052 0.707696 rpy=0 0 0 -> xyz=-2.56148 -1.8052 0.707696 rpy=0 0 0
- joint Cat_395_Part_11_Joint: origin xyz=-0.599 -0.350 -2.289 rpy=0 0 0 -> xyz=0.599 0.350 -2.289 rpy=0 0 0
- joint Cat_395_Part_12_Joint: origin xyz=-0.719 0.000 0.036 rpy=0 0 0 -> xyz=0.719 0.0 0.036 rpy=0 0 0
- joint Cat_395_Track_Left_Joint: origin xyz=-0.02904 -1.709747 0.764672 rpy=0 0 0 -> xyz=-0.02904 1.709747 0.764672 rpy=0 0 0
- joint Cat_395_Track_Right_Joint: origin xyz=-0.02904 1.709747 0.764672 rpy=0 0 0 -> xyz=-0.02904 -1.709747 0.764672 rpy=0 0 0
- joint Cat_395_Wheel_Left_Joint: origin xyz=-2.65099 -1.70966 0.707697 rpy=0 0 0 -> xyz=2.65099 1.70966 0.707697 rpy=0 0 0
- joint Cat_395_Wheel_Right_Joint: origin xyz=-2.65099 1.70966 0.707697 rpy=0 0 0 -> xyz=2.65099 -1.70966 0.707697 rpy=0 0 0

File: excavator/description/urdf/excavator.xacro (robot description, xacro)
@@ -4,22 +4,28 @@
     <link name="${prefix}Base">
       <visual>
-        <origin xyz="0.0 0.0 0.793384" rpy="0 0 ${pi}" />
-        <geometry>
-          <mesh filename="package://construction_vehicles/excavator/description/meshes/visual/Base_Without_Wheels_Rotate_180.dae" />
-        </geometry>
-      </visual>
-      <collision>
-        <origin xyz="0.068918 0.0 1.38521" rpy="0 0 0" />
-        <geometry>
-          <box size="2.85584 4.44524 0.684194" />
-        </geometry>
-      </collision>
+        <origin xyz="0.0 0.0 0.793384" rpy="0 0 0" />
+        <geometry>
+          <mesh filename="package://construction_vehicles/excavator/description/meshes/visual/Base_Without_Wheels.dae" />
+        </geometry>
+      </visual>
     </link>
     <joint name="${prefix}Track_Left_Joint" type="fixed">
+      <origin xyz="-0.02904 1.709747 0.764672" rpy="0 0 0" />
+      <parent link="${prefix}Base" />
+      <child link="${prefix}Track_Left" />
+    </joint>
+    <link name="${prefix}Track_Left">
+      <visual>
+        <geometry>
+          <mesh filename="package://construction_vehicles/excavator/description/meshes/visual/Track.dae" />
+        </geometry>
+      </visual>
+    </link>
+    <joint name="${prefix}Track_Right_Joint" type="fixed">
       <origin xyz="-0.02904 -1.709747 0.764672" rpy="0 0 0" />
       <parent link="${prefix}Base" />
-      <child link="${prefix}Track_Left" />
-    </joint>
-    <link name="${prefix}Track_Left">
+      <child link="${prefix}Track_Right" />
+    </joint>
+    <link name="${prefix}Track_Right">
       <visual>
         <geometry>
@@ -27,29 +33,7 @@
         </geometry>
       </visual>
-      <collision>
-        <geometry>
-          <box size="6.6022 0.757722 1.57115" />
-        </geometry>
-      </collision>
-    </link>
-    <joint name="${prefix}Track_Right_Joint" type="fixed">
-      <origin xyz="-0.02904 1.709747 0.764672" rpy="0 0 0" />
-      <parent link="${prefix}Base" />
-      <child link="${prefix}Track_Right" />
-    </joint>
-    <link name="${prefix}Track_Right">
-      <visual>
-        <geometry>
-          <mesh filename="package://construction_vehicles/excavator/description/meshes/visual/Track.dae" />
-        </geometry>
-      </visual>
-      <collision>
-        <geometry>
-          <box size="6.6022 0.757722 1.57115" />
-        </geometry>
-      </collision>
     </link>
     <joint name="${prefix}Motor_Left_Joint" type="continuous">
-      <origin xyz="2.56148 -1.8052 0.707696" rpy="0 0 0" />
+      <origin xyz="-2.56148 1.8052 0.707696" rpy="0 0 0" />
       <parent link="${prefix}Base" />
       <child link="${prefix}Motor_Left" />
@@ -62,12 +46,7 @@
         </geometry>
       </visual>
-      <collision>
-        <geometry>
-          <cylinder radius="0.522574" length="0.531622" />
-        </geometry>
-      </collision>
     </link>
     <joint name="${prefix}Motor_Right_Joint" type="continuous">
-      <origin xyz="2.56148 1.8052 0.707696" rpy="0 0 0" />
+      <origin xyz="-2.56148 -1.8052 0.707696" rpy="0 0 0" />
       <parent link="${prefix}Base" />
       <child link="${prefix}Motor_Right" />
@@ -80,12 +59,7 @@
         </geometry>
       </visual>
-      <collision>
-        <geometry>
-          <cylinder radius="0.522574" length="0.531622" />
-        </geometry>
-      </collision>
     </link>
     <joint name="${prefix}Wheel_Left_Joint" type="continuous">
-      <origin xyz="-2.65099 -1.70966 0.707697" rpy="0 0 0" />
+      <origin xyz="2.65099 1.70966 0.707697" rpy="0 0 0" />
       <parent link="${prefix}Base" />
       <child link="${prefix}Wheel_Left" />
@@ -98,12 +72,7 @@
         </geometry>
       </visual>
-      <collision>
-        <geometry>
-          <cylinder radius="0.46" length="0.177212" />
-        </geometry>
-      </collision>
     </link>
     <joint name="${prefix}Wheel_Right_Joint" type="continuous">
-      <origin xyz="-2.65099 1.70966 0.707697" rpy="0 0 0" />
+      <origin xyz="2.65099 -1.70966 0.707697" rpy="0 0 0" />
       <parent link="${prefix}Base" />
       <child link="${prefix}Wheel_Right" />
@@ -116,9 +85,4 @@
         </geometry>
       </visual>
-      <collision>
-        <geometry>
-          <cylinder radius="0.46" length="0.177212" />
-        </geometry>
-      </collision>
     </link>
     <joint name="Cat_395_Cabin_Joint" type="revolute">
@@ -135,13 +99,7 @@
         </geometry>
       </visual>
-      <collision>
-        <origin xyz="1.24333 0.0 1.98011" rpy="0 0 0" />
-        <geometry>
-          <box size="6.92858 4.5 2.0914" />
-        </geometry>
-      </collision>
     </link>
     <joint name="${prefix}Door_Joint" type="revolute">
-      <origin xyz="-0.9692 -1.757323 2.610876" rpy="0 0 0" />
+      <origin xyz="0.9692 1.757323 2.610876" rpy="0 0 0" />
       <parent link="${prefix}Cabin" />
       <child link="${prefix}Door" />
@@ -155,12 +113,7 @@
         </geometry>
       </visual>
-      <collision>
-        <geometry>
-          <mesh filename="package://construction_vehicles/excavator/description/meshes/collision/Door.stl" />
-        </geometry>
-      </collision>
     </link>
     <joint name="${prefix}Boom_Joint" type="continuous">
-      <origin xyz="-0.340 0.0 2.047" rpy="0 0 0" />
+      <origin xyz="0.340 0.0 2.047" rpy="0 0 0" />
       <parent link="${prefix}Cabin" />
       <child link="${prefix}Boom" />
@@ -173,12 +126,7 @@
         </geometry>
       </visual>
-      <collision>
-        <geometry>
-          <mesh filename="package://construction_vehicles/excavator/description/meshes/collision/Boom_No_Wires.stl" />
-        </geometry>
-      </collision>
     </link>
     <joint name="${prefix}Boom_Cylinder_1_Joint" type="continuous">
-      <origin xyz="-1.269 0.0 1.167" rpy="0 ${-34/180 * pi} 0" />
+      <origin xyz="1.269 0.0 1.167" rpy="0 ${34/180 * pi} 0" />
       <parent link="${prefix}Cabin" />
       <child link="${prefix}Boom_Cylinder_1" />
@@ -187,27 +135,15 @@
     <link name="${prefix}Boom_Cylinder_1">
       <visual>
+        <origin xyz="0.0 0.506 0.0" rpy="0 0 0" />
+        <geometry>
+          <mesh filename="package://construction_vehicles/excavator/description/meshes/visual/Boom_Cylinder_Left_1.dae" />
+        </geometry>
+      </visual>
+      <visual>
         <origin xyz="0.0 -0.506 0.0" rpy="0 0 0" />
         <geometry>
-          <mesh filename="package://construction_vehicles/excavator/description/meshes/visual/Boom_Cylinder_Left_1.dae" />
-        </geometry>
-      </visual>
-      <visual>
-        <origin xyz="0.0 0.506 0.0" rpy="0 0 0" />
-        <geometry>
           <mesh filename="package://construction_vehicles/excavator/description/meshes/visual/Boom_Cylinder_Right_1.dae" />
         </geometry>
       </visual>
-      <collision>
-        <origin xyz="0.0 -0.506 1.09389" rpy="0 0 0" />
-        <geometry>
-          <cylinder radius="0.271748" length="2.46036" />
-        </geometry>
-      </collision>
-      <collision>
-        <origin xyz="0.0 0.506 1.09389" rpy="0 0 0" />
-        <geometry>
-          <cylinder radius="0.271748" length="2.46036" />
-        </geometry>
-      </collision>
     </link>
     <joint name="${prefix}Boom_Cylinder_2_Joint" type="prismatic">
@@ -220,30 +156,18 @@
     <link name="${prefix}Boom_Cylinder_2">
       <visual>
+        <origin xyz="0.0 0.506 0.0" rpy="0 0 0" />
+        <geometry>
+          <mesh filename="package://construction_vehicles/excavator/description/meshes/visual/Boom_Cylinder_Left_2.dae" />
+        </geometry>
+      </visual>
+      <visual>
         <origin xyz="0.0 -0.506 0.0" rpy="0 0 0" />
         <geometry>
-          <mesh filename="package://construction_vehicles/excavator/description/meshes/visual/Boom_Cylinder_Left_2.dae" />
-        </geometry>
-      </visual>
-      <visual>
-        <origin xyz="0.0 0.506 0.0" rpy="0 0 0" />
-        <geometry>
           <mesh filename="package://construction_vehicles/excavator/description/meshes/visual/Boom_Cylinder_Right_2.dae" />
         </geometry>
       </visual>
-      <collision>
-        <origin xyz="0.0 -0.506 -1.11271" rpy="0 0 0" />
-        <geometry>
-          <cylinder radius="0.120975" length="2.46738" />
-        </geometry>
-      </collision>
-      <collision>
-        <origin xyz="0.0 0.506 -1.11271" rpy="0 0 0" />
-        <geometry>
-          <cylinder radius="0.120975" length="2.46738" />
-        </geometry>
-      </collision>
     </link>
     <joint name="${prefix}Arm_Cylinder_1_Joint" type="continuous">
-      <origin xyz="-2.605 0.000 3.306" rpy="0 ${-81/180 * pi} 0" />
+      <origin xyz="2.605 0.000 3.306" rpy="0 ${81/180 * pi} 0" />
       <parent link="${prefix}Boom" />
       <child link="${prefix}Arm_Cylinder_1" />
@@ -256,10 +180,4 @@
         </geometry>
       </visual>
-      <collision>
-        <origin xyz="0.0 0.0 1.4316" rpy="0 0 0" />
-        <geometry>
-          <cylinder radius="0.262538" length="3.1358" />
-        </geometry>
-      </collision>
     </link>
     <joint name="${prefix}Arm_Cylinder_2_Joint" type="prismatic">
@@ -276,13 +194,7 @@
         </geometry>
       </visual>
-      <collision>
-        <origin xyz="0.0 0.0 -1.09116" rpy="0 0 0" />
-        <geometry>
-          <cylinder radius="0.120975" length="2.42278" />
-        </geometry>
-      </collision>
     </link>
     <joint name="${prefix}Arm_Joint" type="continuous">
-      <origin xyz="-7.002 0.000 2.732" rpy="0 0 0" />
+      <origin xyz="7.002 0.000 2.732" rpy="0 0 0" />
       <parent link="${prefix}Boom" />
       <child link="${prefix}Arm" />
@@ -295,12 +207,7 @@
         </geometry>
       </visual>
-      <collision>
-        <geometry>
-          <mesh filename="package://construction_vehicles/excavator/description/meshes/collision/Arm.stl" />
-        </geometry>
-      </collision>
     </link>
     <joint name="${prefix}Bucket_Cylinder_1_Joint" type="continuous">
-      <origin xyz="-0.999 0.000 1.120" rpy="0 ${8.97/180 * pi} 0" />
+      <origin xyz="0.999 0.000 1.120" rpy="0 ${-8.97/180 * pi} 0" />
       <parent link="${prefix}Arm" />
       <child link="${prefix}Bucket_Cylinder_1" />
@@ -313,10 +220,4 @@
         </geometry>
       </visual>
-      <collision>
-        <origin xyz="0.0 0.0 -1.11" rpy="0 0 0" />
-        <geometry>
-          <cylinder radius="0.173211" length="2.49252" />
-        </geometry>
-      </collision>
     </link>
     <joint name="${prefix}Bucket_Cylinder_2_Joint" type="prismatic">
@@ -333,13 +234,7 @@
         </geometry>
       </visual>
-      <collision>
-        <origin xyz="0.0 0.0 0.583215" rpy="0 0 0" />
-        <geometry>
-          <cylinder radius="0.120975" length="1.408384" />
-        </geometry>
-      </collision>
     </link>
     <joint name="${prefix}Part_11_Joint" type="continuous">
-      <origin xyz="-0.599 -0.350 -2.289" rpy="0 0 0" />
+      <origin xyz="0.599 0.350 -2.289" rpy="0 0 0" />
       <parent link="${prefix}Arm" />
       <child link="${prefix}Part_11" />
@@ -352,12 +247,7 @@
         </geometry>
       </visual>
-      <collision>
-        <geometry>
-          <mesh filename="package://construction_vehicles/excavator/description/meshes/collision/Part_11.stl" />
-        </geometry>
-      </collision>
     </link>
     <joint name="${prefix}Bucket_Joint" type="continuous">
-      <origin xyz="-0.659 0.000 -2.843" rpy="0 0 0" />
+      <origin xyz="0.659 0.0 -2.843" rpy="0 0 0" />
       <parent link="${prefix}Arm" />
       <child link="${prefix}Bucket" />
@@ -370,12 +260,7 @@
         </geometry>
       </visual>
-      <collision>
-        <geometry>
-          <mesh filename="package://construction_vehicles/excavator/description/meshes/collision/Bucket.stl" />
-        </geometry>
-      </collision>
     </link>
     <joint name="${prefix}Part_12_Joint" type="continuous">
-      <origin xyz="-0.719 0.000 0.036" rpy="0 0 0" />
+      <origin xyz="0.719 0.0 0.036" rpy="0 0 0" />
       <parent link="${prefix}Bucket" />
       <child link="${prefix}Part_12" />
@@ -388,9 +273,4 @@
         </geometry>
       </visual>
-      <collision>
-        <geometry>
-          <mesh filename="package://construction_vehicles/excavator/description/meshes/collision/Part_12.stl" />
-        </geometry>
-      </collision>
     </link>
   </xacro:macro>
