Commit message: Conform vehicles

File: excavator/description/urdf/excavator.urdf (robot description, URDF)
Before this commit: robot excavator, 20 links, 19 joints
Links:
- removed link Cat_395_Arm_Cylinder_1
- removed link Cat_395_Arm_Cylinder_2
- removed link Cat_395_Boom_Cylinder_1
- removed link Cat_395_Boom_Cylinder_2
- removed link Cat_395_Bucket_Cylinder_1
- removed link Cat_395_Bucket_Cylinder_2
- removed link Cat_395_Motor_Left
- removed link Cat_395_Motor_Right
- removed link Cat_395_Part_11
- removed link Cat_395_Part_12
- removed link Cat_395_Track_Left
- removed link Cat_395_Track_Right
- removed link Cat_395_Wheel_Left
- removed link Cat_395_Wheel_Right
- added link Cat_395_ArmCylinder1; visual mesh filename=package://construction_vehicles/excavator/description/meshe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
- added link Cat_395_ArmCylinder2; visual mesh filename=package://construction_vehicles/excavator/description/meshe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
- added link Cat_395_BoomCylinder1; visual mesh filename=package://construction_vehicles/excavator/description/meshe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; visual mesh filename=package://construction_vehicles/excavator/description/meshe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
- added link Cat_395_BoomCylinder2; visual mesh filename=package://construction_vehicles/excavator/description/meshe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; visual mesh filename=package://construction_vehicles/excavator/description/meshe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
- added link Cat_395_BucketCylinder1; visual mesh filename=package://construction_vehicles/excavator/description/meshe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
- added link Cat_395_BucketCylinder2; visual mesh filename=package://construction_vehicles/excavator/description/meshe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
- added link Cat_395_MotorLeft; visual mesh filename=package://construction_vehicles/excavator/description/meshe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
- added link Cat_395_MotorRight; visual mesh filename=package://construction_vehicles/excavator/description/meshe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
- added link Cat_395_Part11; visual mesh filename=package://construction_vehicles/excavator/description/meshe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
- added link Cat_395_Part12; visual mesh filename=package://construction_vehicles/excavator/description/meshe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
- added link Cat_395_TrackLeft; visual mesh filename=package://construction_vehicles/excavator/description/meshe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
- added link Cat_395_TrackRight; visual mesh filename=package://construction_vehicles/excavator/description/meshe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
- added link Cat_395_WheelLeft; visual mesh filename=package://construction_vehicles/excavator/description/meshe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
- added link Cat_395_WheelRight; visual mesh filename=package://construction_vehicles/excavator/description/meshe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
Joints:
- removed joint Cat_395_Arm_Cylinder_1_Joint
- removed joint Cat_395_Arm_Cylinder_2_Joint
- removed joint Cat_395_Boom_Cylinder_1_Joint
- removed joint Cat_395_Boom_Cylinder_2_Joint
- removed joint Cat_395_Bucket_Cylinder_1_Joint
- removed joint Cat_395_Bucket_Cylinder_2_Joint
- removed joint Cat_395_Motor_Left_Joint
- removed joint Cat_395_Motor_Right_Joint
- removed joint Cat_395_Part_11_Joint
- removed joint Cat_395_Part_12_Joint
- removed joint Cat_395_Track_Left_Joint
- removed joint Cat_395_Track_Right_Joint
- removed joint Cat_395_Wheel_Left_Joint
- removed joint Cat_395_Wheel_Right_Joint
- added joint Cat_395_ArmCylinder1_Joint: type continuous, parent Cat_395_Boom, child Cat_395_ArmCylinder1, origin xyz=2.605 0.000 3.306 rpy=0 1.413716694115407 0, axis 0 1 0
- added joint Cat_395_ArmCylinder2_Joint: type prismatic, parent Cat_395_ArmCylinder1, child Cat_395_ArmCylinder2, origin xyz=0.0 0.0 4.76576 rpy=0 0 0, axis 0 0 1, limit lower=-1.6 upper=0.38 effort=1000.0 velocity=1000.0
- added joint Cat_395_BoomCylinder1_Joint: type continuous, parent Cat_395_Cabin, child Cat_395_BoomCylinder1, origin xyz=1.269 0.0 1.167 rpy=0 0.593411945678072 0, axis 0 1 0
- added joint Cat_395_BoomCylinder2_Joint: type prismatic, parent Cat_395_BoomCylinder1, child Cat_395_BoomCylinder2, origin xyz=0.0 0.0 4.13344 rpy=0 0 0, axis 0 0 1, limit lower=-1.70 upper=0.31 effort=1000.0 velocity=1000.0
- added joint Cat_395_BucketCylinder1_Joint: type continuous, parent Cat_395_Arm, child Cat_395_BucketCylinder1, origin xyz=0.999 0.000 1.120 rpy=0 -0.15655603390389136 0, axis 0 1 0
- added joint Cat_395_BucketCylinder2_Joint: type prismatic, parent Cat_395_BucketCylinder1, child Cat_395_BucketCylinder2, origin xyz=0.0 0.0 -3.1066 rpy=0 0 0, axis 0 0 1, limit lower=-0.41 upper=0.57 effort=1000.0 velocity=1000.0
- added joint Cat_395_MotorLeft_Joint: type continuous, parent Cat_395_Base, child Cat_395_MotorLeft, origin xyz=-2.56148 1.8052 0.707696 rpy=0 0 0, axis 0 -1 0
- added joint Cat_395_MotorRight_Joint: type continuous, parent Cat_395_Base, child Cat_395_MotorRight, origin xyz=-2.56148 -1.8052 0.707696 rpy=0 0 0, axis 0 -1 0
- added joint Cat_395_Part11_Joint: type continuous, parent Cat_395_Arm, child Cat_395_Part11, origin xyz=0.599 0.350 -2.289 rpy=0 0 0, axis 0 1 0
- added joint Cat_395_Part12_Joint: type continuous, parent Cat_395_Bucket, child Cat_395_Part12, origin xyz=0.719 0.0 0.036 rpy=0 0 0, axis 0 1 0
- added joint Cat_395_TrackLeft_Joint: type fixed, parent Cat_395_Base, child Cat_395_TrackLeft, origin xyz=-0.02904 1.709747 0.764672 rpy=0 0 0
- added joint Cat_395_TrackRight_Joint: type fixed, parent Cat_395_Base, child Cat_395_TrackRight, origin xyz=-0.02904 -1.709747 0.764672 rpy=0 0 0
- added joint Cat_395_WheelLeft_Joint: type continuous, parent Cat_395_Base, child Cat_395_WheelLeft, origin xyz=2.65099 1.70966 0.707697 rpy=0 0 0, axis 0 -1 0
- added joint Cat_395_WheelRight_Joint: type continuous, parent Cat_395_Base, child Cat_395_WheelRight, origin xyz=2.65099 -1.70966 0.707697 rpy=0 0 0, axis 0 -1 0

File: excavator/description/urdf/excavator.xacro (robot description, xacro)
@@ -6,14 +6,14 @@
         <origin xyz="0.0 0.0 0.793384" rpy="0 0 0" />
         <geometry>
-          <mesh filename="package://construction_vehicles/excavator/description/meshes/visual/Base_Without_Wheels.dae" />
-        </geometry>
-      </visual>
-    </link>
-    <joint name="${prefix}Track_Left_Joint" type="fixed">
+          <mesh filename="package://construction_vehicles/excavator/description/meshes/visual/BaseWithoutWheels.dae" />
+        </geometry>
+      </visual>
+    </link>
+    <joint name="${prefix}TrackLeft_Joint" type="fixed">
       <origin xyz="-0.02904 1.709747 0.764672" rpy="0 0 0" />
       <parent link="${prefix}Base" />
-      <child link="${prefix}Track_Left" />
-    </joint>
-    <link name="${prefix}Track_Left">
+      <child link="${prefix}TrackLeft" />
+    </joint>
+    <link name="${prefix}TrackLeft">
       <visual>
         <geometry>
@@ -22,10 +22,10 @@
       </visual>
     </link>
-    <joint name="${prefix}Track_Right_Joint" type="fixed">
+    <joint name="${prefix}TrackRight_Joint" type="fixed">
       <origin xyz="-0.02904 -1.709747 0.764672" rpy="0 0 0" />
       <parent link="${prefix}Base" />
-      <child link="${prefix}Track_Right" />
-    </joint>
-    <link name="${prefix}Track_Right">
+      <child link="${prefix}TrackRight" />
+    </joint>
+    <link name="${prefix}TrackRight">
       <visual>
         <geometry>
@@ -34,37 +34,37 @@
       </visual>
     </link>
-    <joint name="${prefix}Motor_Left_Joint" type="continuous">
+    <joint name="${prefix}MotorLeft_Joint" type="continuous">
       <origin xyz="-2.56148 1.8052 0.707696" rpy="0 0 0" />
       <parent link="${prefix}Base" />
-      <child link="${prefix}Motor_Left" />
-      <axis xyz="0 -1 0" />
-    </joint>
-    <link name="${prefix}Motor_Left">
-      <visual>
-        <geometry>
-          <mesh filename="package://construction_vehicles/excavator/description/meshes/visual/Motor_Left.dae" />
-        </geometry>
-      </visual>
-    </link>
-    <joint name="${prefix}Motor_Right_Joint" type="continuous">
+      <child link="${prefix}MotorLeft" />
+      <axis xyz="0 -1 0" />
+    </joint>
+    <link name="${prefix}MotorLeft">
+      <visual>
+        <geometry>
+          <mesh filename="package://construction_vehicles/excavator/description/meshes/visual/MotorLeft.dae" />
+        </geometry>
+      </visual>
+    </link>
+    <joint name="${prefix}MotorRight_Joint" type="continuous">
       <origin xyz="-2.56148 -1.8052 0.707696" rpy="0 0 0" />
       <parent link="${prefix}Base" />
-      <child link="${prefix}Motor_Right" />
-      <axis xyz="0 -1 0" />
-    </joint>
-    <link name="${prefix}Motor_Right">
-      <visual>
-        <geometry>
-          <mesh filename="package://construction_vehicles/excavator/description/meshes/visual/Motor_Right.dae" />
-        </geometry>
-      </visual>
-    </link>
-    <joint name="${prefix}Wheel_Left_Joint" type="continuous">
+      <child link="${prefix}MotorRight" />
+      <axis xyz="0 -1 0" />
+    </joint>
+    <link name="${prefix}MotorRight">
+      <visual>
+        <geometry>
+          <mesh filename="package://construction_vehicles/excavator/description/meshes/visual/MotorRight.dae" />
+        </geometry>
+      </visual>
+    </link>
+    <joint name="${prefix}WheelLeft_Joint" type="continuous">
       <origin xyz="2.65099 1.70966 0.707697" rpy="0 0 0" />
       <parent link="${prefix}Base" />
-      <child link="${prefix}Wheel_Left" />
-      <axis xyz="0 -1 0" />
-    </joint>
-    <link name="${prefix}Wheel_Left">
+      <child link="${prefix}WheelLeft" />
+      <axis xyz="0 -1 0" />
+    </joint>
+    <link name="${prefix}WheelLeft">
       <visual>
         <geometry>
@@ -73,11 +73,11 @@
       </visual>
     </link>
-    <joint name="${prefix}Wheel_Right_Joint" type="continuous">
+    <joint name="${prefix}WheelRight_Joint" type="continuous">
       <origin xyz="2.65099 -1.70966 0.707697" rpy="0 0 0" />
       <parent link="${prefix}Base" />
-      <child link="${prefix}Wheel_Right" />
-      <axis xyz="0 -1 0" />
-    </joint>
-    <link name="${prefix}Wheel_Right">
+      <child link="${prefix}WheelRight" />
+      <axis xyz="0 -1 0" />
+    </joint>
+    <link name="${prefix}WheelRight">
       <visual>
         <geometry>
@@ -96,5 +96,5 @@
       <visual>
         <geometry>
-          <mesh filename="package://construction_vehicles/excavator/description/meshes/visual/Cabin_No_Wires.dae" />
+          <mesh filename="package://construction_vehicles/excavator/description/meshes/visual/CabinNoWires.dae" />
         </geometry>
       </visual>
@@ -123,19 +123,19 @@
       <visual>
         <geometry>
-          <mesh filename="package://construction_vehicles/excavator/description/meshes/visual/Boom_No_Wires.dae" />
-        </geometry>
-      </visual>
-    </link>
-    <joint name="${prefix}Boom_Cylinder_1_Joint" type="continuous">
+          <mesh filename="package://construction_vehicles/excavator/description/meshes/visual/BoomNoWires.dae" />
+        </geometry>
+      </visual>
+    </link>
+    <joint name="${prefix}BoomCylinder1_Joint" type="continuous">
       <origin xyz="1.269 0.0 1.167" rpy="0 ${34/180 * pi} 0" />
       <parent link="${prefix}Cabin" />
-      <child link="${prefix}Boom_Cylinder_1" />
-      <axis xyz="0 1 0" />
-    </joint>
-    <link name="${prefix}Boom_Cylinder_1">
+      <child link="${prefix}BoomCylinder1" />
+      <axis xyz="0 1 0" />
+    </joint>
+    <link name="${prefix}BoomCylinder1">
       <visual>
         <origin xyz="0.0 0.506 0.0" rpy="0 0 0" />
         <geometry>
-          <mesh filename="package://construction_vehicles/excavator/description/meshes/visual/Boom_Cylinder_Left_1.dae" />
+          <mesh filename="package://construction_vehicles/excavator/description/meshes/visual/BoomCylinderLeft1.dae" />
         </geometry>
       </visual>
@@ -143,20 +143,20 @@
         <origin xyz="0.0 -0.506 0.0" rpy="0 0 0" />
         <geometry>
-          <mesh filename="package://construction_vehicles/excavator/description/meshes/visual/Boom_Cylinder_Right_1.dae" />
-        </geometry>
-      </visual>
-    </link>
-    <joint name="${prefix}Boom_Cylinder_2_Joint" type="prismatic">
+          <mesh filename="package://construction_vehicles/excavator/description/meshes/visual/BoomCylinderRight1.dae" />
+        </geometry>
+      </visual>
+    </link>
+    <joint name="${prefix}BoomCylinder2_Joint" type="prismatic">
       <origin xyz="0.0 0.0 4.13344" rpy="0 0 0" />
-      <parent link="${prefix}Boom_Cylinder_1" />
-      <child link="${prefix}Boom_Cylinder_2" />
+      <parent link="${prefix}BoomCylinder1" />
+      <child link="${prefix}BoomCylinder2" />
       <axis xyz="0 0 1" />
       <limit lower="-1.70" upper="0.31" effort="1000.0" velocity="1000.0" />
     </joint>
-    <link name="${prefix}Boom_Cylinder_2">
+    <link name="${prefix}BoomCylinder2">
       <visual>
         <origin xyz="0.0 0.506 0.0" rpy="0 0 0" />
         <geometry>
-          <mesh filename="package://construction_vehicles/excavator/description/meshes/visual/Boom_Cylinder_Left_2.dae" />
+          <mesh filename="package://construction_vehicles/excavator/description/meshes/visual/BoomCylinderLeft2.dae" />
         </geometry>
       </visual>
@@ -164,32 +164,32 @@
         <origin xyz="0.0 -0.506 0.0" rpy="0 0 0" />
         <geometry>
-          <mesh filename="package://construction_vehicles/excavator/description/meshes/visual/Boom_Cylinder_Right_2.dae" />
-        </geometry>
-      </visual>
-    </link>
-    <joint name="${prefix}Arm_Cylinder_1_Joint" type="continuous">
+          <mesh filename="package://construction_vehicles/excavator/description/meshes/visual/BoomCylinderRight2.dae" />
+        </geometry>
+      </visual>
+    </link>
+    <joint name="${prefix}ArmCylinder1_Joint" type="continuous">
       <origin xyz="2.605 0.000 3.306" rpy="0 ${81/180 * pi} 0" />
       <parent link="${prefix}Boom" />
-      <child link="${prefix}Arm_Cylinder_1" />
-      <axis xyz="0 1 0" />
-    </joint>
-    <link name="${prefix}Arm_Cylinder_1">
-      <visual>
-        <geometry>
-          <mesh filename="package://construction_vehicles/excavator/description/meshes/visual/Arm_Cylinder_1.dae" />
-        </geometry>
-      </visual>
-    </link>
-    <joint name="${prefix}Arm_Cylinder_2_Joint" type="prismatic">
+      <child link="${prefix}ArmCylinder1" />
+      <axis xyz="0 1 0" />
+    </joint>
+    <link name="${prefix}ArmCylinder1">
+      <visual>
+        <geometry>
+          <mesh filename="package://construction_vehicles/excavator/description/meshes/visual/ArmCylinder1.dae" />
+        </geometry>
+      </visual>
+    </link>
+    <joint name="${prefix}ArmCylinder2_Joint" type="prismatic">
       <origin xyz="0.0 0.0 4.76576" rpy="0 0 0" />
-      <parent link="${prefix}Arm_Cylinder_1" />
-      <child link="${prefix}Arm_Cylinder_2" />
+      <parent link="${prefix}ArmCylinder1" />
+      <child link="${prefix}ArmCylinder2" />
       <axis xyz="0 0 1" />
       <limit lower="-1.6" upper="0.38" effort="1000.0" velocity="1000.0" />
     </joint>
-    <link name="${prefix}Arm_Cylinder_2">
-      <visual>
-        <geometry>
-          <mesh filename="package://construction_vehicles/excavator/description/meshes/visual/Arm_Cylinder_2.dae" />
+    <link name="${prefix}ArmCylinder2">
+      <visual>
+        <geometry>
+          <mesh filename="package://construction_vehicles/excavator/description/meshes/visual/ArmCylinder2.dae" />
         </geometry>
       </visual>
@@ -208,41 +208,41 @@
       </visual>
     </link>
-    <joint name="${prefix}Bucket_Cylinder_1_Joint" type="continuous">
+    <joint name="${prefix}BucketCylinder1_Joint" type="continuous">
       <origin xyz="0.999 0.000 1.120" rpy="0 ${-8.97/180 * pi} 0" />
       <parent link="${prefix}Arm" />
-      <child link="${prefix}Bucket_Cylinder_1" />
-      <axis xyz="0 1 0" />
-    </joint>
-    <link name="${prefix}Bucket_Cylinder_1">
-      <visual>
-        <geometry>
-          <mesh filename="package://construction_vehicles/excavator/description/meshes/visual/Bucket_Cylinder_1.dae" />
-        </geometry>
-      </visual>
-    </link>
-    <joint name="${prefix}Bucket_Cylinder_2_Joint" type="prismatic">
+      <child link="${prefix}BucketCylinder1" />
+      <axis xyz="0 1 0" />
+    </joint>
+    <link name="${prefix}BucketCylinder1">
+      <visual>
+        <geometry>
+          <mesh filename="package://construction_vehicles/excavator/description/meshes/visual/BucketCylinder1.dae" />
+        </geometry>
+      </visual>
+    </link>
+    <joint name="${prefix}BucketCylinder2_Joint" type="prismatic">
       <origin xyz="0.0 0.0 -3.1066" rpy="0 0 0" />
-      <parent link="${prefix}Bucket_Cylinder_1" />
-      <child link="${prefix}Bucket_Cylinder_2" />
+      <parent link="${prefix}BucketCylinder1" />
+      <child link="${prefix}BucketCylinder2" />
       <axis xyz="0 0 1" />
       <limit lower="-0.41" upper="0.57" effort="1000.0" velocity="1000.0" />
     </joint>
-    <link name="${prefix}Bucket_Cylinder_2">
-      <visual>
-        <geometry>
-          <mesh filename="package://construction_vehicles/excavator/description/meshes/visual/Bucket_Cylinder_2.dae" />
-        </geometry>
-      </visual>
-    </link>
-    <joint name="${prefix}Part_11_Joint" type="continuous">
+    <link name="${prefix}BucketCylinder2">
+      <visual>
+        <geometry>
+          <mesh filename="package://construction_vehicles/excavator/description/meshes/visual/BucketCylinder2.dae" />
+        </geometry>
+      </visual>
+    </link>
+    <joint name="${prefix}Part11_Joint" type="continuous">
       <origin xyz="0.599 0.350 -2.289" rpy="0 0 0" />
       <parent link="${prefix}Arm" />
-      <child link="${prefix}Part_11" />
-      <axis xyz="0 1 0" />
-    </joint>
-    <link name="${prefix}Part_11">
-      <visual>
-        <geometry>
-          <mesh filename="package://construction_vehicles/excavator/description/meshes/visual/Part_11.dae" />
+      <child link="${prefix}Part11" />
+      <axis xyz="0 1 0" />
+    </joint>
+    <link name="${prefix}Part11">
+      <visual>
+        <geometry>
+          <mesh filename="package://construction_vehicles/excavator/description/meshes/visual/Part11.dae" />
         </geometry>
       </visual>
@@ -261,14 +261,14 @@
       </visual>
     </link>
-    <joint name="${prefix}Part_12_Joint" type="continuous">
+    <joint name="${prefix}Part12_Joint" type="continuous">
       <origin xyz="0.719 0.0 0.036" rpy="0 0 0" />
       <parent link="${prefix}Bucket" />
-      <child link="${prefix}Part_12" />
-      <axis xyz="0 1 0" />
-    </joint>
-    <link name="${prefix}Part_12">
-      <visual>
-        <geometry>
-          <mesh filename="package://construction_vehicles/excavator/description/meshes/visual/Part_12.dae" />
+      <child link="${prefix}Part12" />
+      <axis xyz="0 1 0" />
+    </joint>
+    <link name="${prefix}Part12">
+      <visual>
+        <geometry>
+          <mesh filename="package://construction_vehicles/excavator/description/meshes/visual/Part12.dae" />
         </geometry>
       </visual>
