Commit message: Add cat 6015B and fix cat 395

File: excavator/description/urdf/excavator.xacro (robot description, xacro)
@@ -152,5 +152,5 @@
       <child link="${prefix}BoomCylinder2" />
       <axis xyz="0 0 1" />
-      <limit lower="-1.70" upper="0.31" effort="1000.0" velocity="1000.0" />
+      <limit lower="-1.20" upper="1.10" effort="1000.0" velocity="1000.0" />
     </joint>
     <link name="${prefix}BoomCylinder2">
@@ -186,5 +186,5 @@
       <child link="${prefix}ArmCylinder2" />
       <axis xyz="0 0 1" />
-      <limit lower="-1.6" upper="0.38" effort="1000.0" velocity="1000.0" />
+      <limit lower="-1.60" upper="0.80" effort="1000.0" velocity="1000.0" />
     </joint>
     <link name="${prefix}ArmCylinder2">
@@ -226,5 +226,5 @@
       <child link="${prefix}BucketCylinder2" />
       <axis xyz="0 0 1" />
-      <limit lower="-0.41" upper="0.57" effort="1000.0" velocity="1000.0" />
+      <limit lower="-0.60" upper="0.20" effort="1000.0" velocity="1000.0" />
     </joint>
     <link name="${prefix}BucketCylinder2">
